Commit message: zmieniony model kolizji kol

File: src/boxygo/urdf/6_wheel_robot_v3.urdf.xacro (robot description, xacro)
@@ -8,11 +8,12 @@
   <xacro:property name="wheel_width" value="0.05"/>
   <xacro:property name="wheel_gap" value="0.35"/>
-  <xacro:property name="wheel_y_offset" value="${0.5 * body_width + 0.009}"/>
+  <xacro:property name="wheel_y_offset" value="${0.5 * body_width + 0.5 * wheel_width}"/>
   <xacro:property name="wheel_mass" value="3.0"/>
   <xacro:property name="pkg_path" value="$(find boxygo)"/>
   <!-- Materiały -->
   <material name="black"><color rgba="0 0 0 1"/></material>
-  <material name="white"><color rgba="0.7 0.7 0.7 0.5"/></material>
-  <material name="grey"><color rgba="0.5 0.5 0.5 1"/></material>
+  <material name="blue"><color rgba="0 0 1 1"/></material>
+  <material name="red"><color rgba="1 0 0 1"/></material>
+  <material name="white"><color rgba="1 1 1 1"/></material>
   <!-- Korpus -->
   <link name="base_link">
@@ -21,5 +22,5 @@
         <box size="${body_length} ${body_width} ${body_height}"/>
       </geometry>
-      <material name="white"/>
+      <material name="blue"/>
     </visual>
     <collision>
@@ -34,26 +35,31 @@
   </link>
   <!-- Makro koła -->
-  <xacro:macro name="wheel" params="side wheel_side_sign joint_sign index x_offset">
-    <xacro:property name="ixx" value="${(1.0/12.0) * wheel_mass * (3 * wheel_radius**2 + wheel_width**2)}"/>
+  <xacro:macro name="wheel" params="side index x_offset">
+    <xacro:property name="wheel_side_sign" value="${1 if side == 'left' else -1}"/>
+    <xacro:property name=
+"ixx" value="${(1.0/12.0) * wheel_mass * (3 * wheel_radius**2 + wheel_width**2)}"/>
     <xacro:property name="izz" value="${0.5 * wheel_mass * wheel_radius**2}"/>
     <link name="${side}_wheel_${index}">
+      <!-- Wizualizacja z pliku STL (bezwzględna ścieżka) -->
+      <visual>
+        <geometry>
+          <mesh filename="/home/jakub/BoxyGo/src/boxygo/meshes/hoverboard_wheel.stl" scale="0.001 0.001  0.001 "/>
+        </geometry>
+        <origin xyz="0 0 0" rpy="1.5707 0 0"/>
+        <material name="black"/>
+      </visual>
+      <!-- Kolizja uproszczona -->
+      <collision>
+        <geometry>
+          <cylinder radius="${wheel_radius}" length="${wheel_width}"/>
+        </geometry>
+        <origin xyz="0 0 0" rpy="1.5707 0 0"/>
+      </collision>
       <inertial>
         <mass value="${wheel_mass}"/>
         <inertia ixx="${ixx}" iyy="${ixx}" izz="${izz}" ixy="0.0" ixz="0.0" iyz="0.0"/>
       </inertial>
-      <visual>
-        <geometry>
-          <mesh filename="${pkg_path}/meshes/hov_wheel_look.stl" scale="0.001 0.001 0.001"/>
-        </geometry>
-        <origin xyz="0 0 0" rpy="0 0 ${wheel_side_sign * math.pi}"/>
-        <material name="grey"/>
-      </visual>
-      <collision>
-        <geometry>
-          <mesh filename="${pkg_path}/meshes/hov_wheel_colision.stl" scale="0.001 0.001 0.001"/>
-        </geometry>
-        <origin xyz="0 0 0" rpy="0 0 ${wheel_side_sign * math.pi}"/>
-      </collision>
     </link>
+    <!-- Tarcie dla Gazebo Classic -->
     <gazebo reference="${side}_wheel_${index}">
       <mu1>1.0</mu1>
@@ -67,5 +73,5 @@
       <parent link="base_link"/>
       <child link="${side}_wheel_${index}"/>
-      <origin xyz="${x_offset} ${joint_sign * wheel_y_offset} ${-0.5 * body_height}" rpy="0 0 0"/>
+      <origin xyz="${x_offset} ${wheel_side_sign * wheel_y_offset} ${-0.5 * body_height}" rpy="0 0 0"/>
       <axis xyz="0 1 0"/>
       <limit effort="10.0" velocity="10.0"/>
@@ -84,32 +90,32 @@
   </xacro:macro>
   <!-- Koła lewe -->
-  <xacro:wheel side="left" wheel_side_sign="0" joint_sign="1" index="1" x_offset="${-wheel_gap}"/>
-  <xacro:wheel side="left" wheel_side_sign="0" joint_sign="1" index="2" x_offset="0"/>
-  <xacro:wheel side="left" wheel_side_sign="0" joint_sign="1" index="3" x_offset="${wheel_gap}"/>
+  <xacro:wheel side="left" index="1" x_offset="${-wheel_gap}"/>
+  <xacro:wheel side="left" index="2" x_offset="0"/>
+  <xacro:wheel side="left" index="3" x_offset="${wheel_gap}"/>
   <!-- Koła prawe -->
-  <xacro:wheel side="right" wheel_side_sign="1" joint_sign="-1" index="1" x_offset="${-wheel_gap}"/>
-  <xacro:wheel side="right" wheel_side_sign="1" joint_sign="-1" index="2" x_offset="0"/>
-  <xacro:wheel side="right" wheel_side_sign="1" joint_sign="-1" index="3" x_offset="${wheel_gap}"/>
+  <xacro:wheel side="right" index="1" x_offset="${-wheel_gap}"/>
+  <xacro:wheel side="right" index="2" x_offset="0"/>
+  <xacro:wheel side="right" index="3" x_offset="${wheel_gap}"/>
   <!-- Gazebo - kolor -->
   <gazebo reference="base_link">
-    <material>Gazebo/White</material>
+    <material>Gazebo/Blue</material>
   </gazebo>
   <gazebo reference="left_wheel_1">
-    <material>Gazebo/Grey</material>
+    <material>Gazebo/Red</material>
   </gazebo>
   <gazebo reference="left_wheel_2">
-    <material>Gazebo/Grey</material>
+    <material>Gazebo/Red</material>
   </gazebo>
   <gazebo reference="left_wheel_3">
-    <material>Gazebo/Grey</material>
+    <material>Gazebo/Red</material>
   </gazebo>
   <gazebo reference="right_wheel_1">
-    <material>Gazebo/Grey</material>
+    <material>Gazebo/Red</material>
   </gazebo>
   <gazebo reference="right_wheel_2">
-    <material>Gazebo/Grey</material>
+    <material>Gazebo/Red</material>
   </gazebo>
   <gazebo reference="right_wheel_3">
-    <material>Gazebo/Grey</material>
+    <material>Gazebo/Red</material>
   </gazebo>
   <!-- Plugin ros2_control -->
