Commit message: update

File: src/boxygo/urdf/6_wheel_robot_v2.urdf.xacro (robot description, xacro)
@@ -46,7 +46,7 @@
       <visual>
         <geometry>
-          <mesh filename="package://${pkg_path}/meshes/hoverboard_wheel.stl" scale="0.001 0.001 0.001"/>
+          <mesh filename="${pkg_path}/meshes/hoverboard_wheel.stl" scale="0.001 0.001 0.001"/>
         </geometry>
-        <origin xyz="0 0 0" rpy="1.5707 0 0"/>
+        <origin xyz="0 0 0" rpy="0 0 0"/>
         <material name="black"/>
       </visual>
@@ -60,7 +60,7 @@
       <collision>
         <geometry>
-          <mesh filename="package://${pkg_path}/meshes/hoverboard_wheel.stl" scale="0.001 0.001 0.001"/>
+          <mesh filename="${pkg_path}/meshes/hoverboard_wheel.stl" scale="0.001 0.001 0.001"/>
         </geometry>
-        <origin xyz="0 0 0" rpy="1.5707 0 0"/>
+        <origin xyz="0 0 0" rpy="0 0 0"/>
       </collision>
     </link>

Commit message: update hoverboard wheels

File: src/boxygo/urdf/6_wheel_robot_v2.urdf.xacro (robot description, xacro)
@@ -8,12 +8,11 @@
   <xacro:property name="wheel_width" value="0.05"/>
   <xacro:property name="wheel_gap" value="0.35"/>
-  <xacro:property name="wheel_y_offset" value="${0.5 * body_width + 0.5 * wheel_width}"/>
+  <xacro:property name="wheel_y_offset" value="${0.5 * body_width + 0.009}"/>
   <xacro:property name="wheel_mass" value="3.0"/>
   <xacro:property name="pkg_path" value="$(find boxygo)"/>
   <!-- Materiały -->
   <material name="black"><color rgba="0 0 0 1"/></material>
-  <material name="blue"><color rgba="0 0 1 1"/></material>
-  <material name="red"><color rgba="1 0 0 1"/></material>
-  <material name="white"><color rgba="1 1 1 1"/></material>
+  <material name="white"><color rgba="0.7 0.7 0.7 0.5"/></material>
+  <material name="grey"><color rgba="0.5 0.5 0.5 1"/></material>
   <!-- Korpus -->
   <link name="base_link">
@@ -22,5 +21,5 @@
         <box size="${body_length} ${body_width} ${body_height}"/>
       </geometry>
-      <material name="blue"/>
+      <material name="white"/>
     </visual>
     <collision>
@@ -35,6 +34,5 @@
   </link>
   <!-- Makro koła -->
-  <xacro:macro name="wheel" params="side index x_offset">
-    <xacro:property name="wheel_side_sign" value="${1 if side == 'left' else -1}"/>
+  <xacro:macro name="wheel" params="side wheel_side_sign joint_sign index x_offset">
     <xacro:property name="ixx" value="${(1.0/12.0) * wheel_mass * (3 * wheel_radius**2 + wheel_width**2)}"/>
     <xacro:property name="izz" value="${0.5 * wheel_mass * wheel_radius**2}"/>
@@ -46,24 +44,16 @@
       <visual>
         <geometry>
-          <mesh filename="${pkg_path}/meshes/hoverboard_wheel.stl" scale="0.001 0.001 0.001"/>
+          <mesh filename="${pkg_path}/meshes/hoverboard_wheel_v2.stl" scale="0.001 0.001 0.001"/>
         </geometry>
-        <origin xyz="0 0 0" rpy="0 0 0"/>
-        <material name="black"/>
-      </visual>
-      <visual name="shaft_visual">
-        <geometry>
-          <cylinder radius="0.015" length="${wheel_radius * 2}"/>
-        </geometry>
-        <origin xyz="0 0 0" rpy="0 0 0"/>
-        <material name="white"/>
+        <origin xyz="0 0 0" rpy="0 0 ${wheel_side_sign * 3.141592}"/>
+        <material name="grey"/>
       </visual>
       <collision>
         <geometry>
-          <mesh filename="${pkg_path}/meshes/hoverboard_wheel.stl" scale="0.001 0.001 0.001"/>
+          <mesh filename="${pkg_path}/meshes/hoverboard_wheel_v2.stl" scale="0.001 0.001 0.001"/>
         </geometry>
-        <origin xyz="0 0 0" rpy="0 0 0"/>
+        <origin xyz="0 0 0" rpy="0 0 ${wheel_side_sign * 3.141592}"/>
       </collision>
     </link>
-    <!-- Tarcie dla Gazebo Classic -->
     <gazebo reference="${side}_wheel_${index}">
       <mu1>1.0</mu1>
@@ -77,5 +67,5 @@
       <parent link="base_link"/>
       <child link="${side}_wheel_${index}"/>
-      <origin xyz="${x_offset} ${wheel_side_sign * wheel_y_offset} ${-0.5 * body_height}" rpy="0 0 0"/>
+      <origin xyz="${x_offset} ${joint_sign * wheel_y_offset} ${-0.5 * body_height}" rpy="0 0 0"/>
       <axis xyz="0 1 0"/>
       <limit effort="10.0" velocity="10.0"/>
@@ -94,32 +84,32 @@
   </xacro:macro>
   <!-- Koła lewe -->
-  <xacro:wheel side="left" index="1" x_offset="${-wheel_gap}"/>
-  <xacro:wheel side="left" index="2" x_offset="0"/>
-  <xacro:wheel side="left" index="3" x_offset="${wheel_gap}"/>
+  <xacro:wheel side="left" wheel_side_sign="1" joint_sign="1" index="1" x_offset="${-wheel_gap}"/>
+  <xacro:wheel side="left" wheel_side_sign="1" joint_sign="1" index="2" x_offset="0"/>
+  <xacro:wheel side="left" wheel_side_sign="1" joint_sign="1" index="3" x_offset="${wheel_gap}"/>
   <!-- Koła prawe -->
-  <xacro:wheel side="right" index="1" x_offset="${-wheel_gap}"/>
-  <xacro:wheel side="right" index="2" x_offset="0"/>
-  <xacro:wheel side="right" index="3" x_offset="${wheel_gap}"/>
+  <xacro:wheel side="right" wheel_side_sign="0" joint_sign="-1" index="1" x_offset="${-wheel_gap}"/>
+  <xacro:wheel side="right" wheel_side_sign="0" joint_sign="-1" index="2" x_offset="0"/>
+  <xacro:wheel side="right" wheel_side_sign="0" joint_sign="-1" index="3" x_offset="${wheel_gap}"/>
   <!-- Gazebo - kolor -->
   <gazebo reference="base_link">
-    <material>Gazebo/Blue</material>
+    <material>Gazebo/White</material>
   </gazebo>
   <gazebo reference="left_wheel_1">
-    <material>Gazebo/Red</material>
+    <material>Gazebo/Grey</material>
   </gazebo>
   <gazebo reference="left_wheel_2">
-    <material>Gazebo/Red</material>
+    <material>Gazebo/Grey</material>
   </gazebo>
   <gazebo reference="left_wheel_3">
-    <material>Gazebo/Red</material>
+    <material>Gazebo/Grey</material>
   </gazebo>
   <gazebo reference="right_wheel_1">
-    <material>Gazebo/Red</material>
+    <material>Gazebo/Grey</material>
   </gazebo>
   <gazebo reference="right_wheel_2">
-    <material>Gazebo/Red</material>
+    <material>Gazebo/Grey</material>
   </gazebo>
   <gazebo reference="right_wheel_3">
-    <material>Gazebo/Red</material>
+    <material>Gazebo/Grey</material>
   </gazebo>
   <!-- Plugin ros2_control -->

Commit message: first lidar & camera

File: src/boxygo/urdf/6_wheel_robot_v2.urdf.xacro (robot description, xacro)
@@ -33,4 +33,105 @@
     </inertial>
   </link>
+    <!-- Kamera -->
+  <link name="depth_camera_link">
+    <visual>
+      <geometry>
+        <box size="0.05 0.05 0.05"/>
+      </geometry>
+      <origin xyz="0 0 0" rpy="0 0 0"/>
+      <material name="black"/>
+    </visual>
+    <collision>
+      <geometry>
+        <box size="0.05 0.05 0.05"/>
+      </geometry>
+    </collision>
+    <inertial>
+      <mass value="0.1"/>
+      <inertia ixx="0.0001" ixy="0.0" ixz="0.0" iyy="0.0001" iyz="0.0" izz="0.0001"/>
+    </inertial>
+  </link>
+  <joint name="depth_camera_joint" type="fixed">
+    <parent link="base_link"/>
+    <child link="depth_camera_link"/>
+    <origin xyz="${body_length/2 + 0.025} 0 ${body_height/2 - 0.025 - 0.05}" rpy="0 0 0"/>
+  </joint>
+  <gazebo reference="depth_camera_link">
+    <sensor name="depth_camera_sensor" type="camera">
+      <always_on>true</always_on>
+      <visualize>true</visualize>
+      <update_rate>30.0</update_rate>
+      <camera>
+        <horizontal_fov>1.39626</horizontal_fov>
+        <image>
+          <width>640</width>
+          <height>480</height>
+          <format>R8G8B8</format>
+        </image>
+        <clip>
+          <near>0.1</near>
+          <far>10.0</far>
+        </clip>
+      </camera>
+      <plugin name="depth_camera_controller" filename="libgazebo_ros_camera.so">
+        <camera_name>depth_camera</camera_name>
+        <frame_name>depth_camera_link</frame_name>
+      </plugin>
+    </sensor>
+  </gazebo>
+    <!-- Lidar 2D -->
+  <link name="lidar_link">
+    <visual>
+      <geometry>
+        <cylinder length="0.05" radius="0.03"/>
+      </geometry>
+      <material name="black"/>
+    </visual>
+    <collision>
+      <geometry>
+        <cylinder length="0.05" radius="0.03"/>
+      </geometry>
+    </collision>
+    <inertial>
+      <mass value="0.2"/>
+      <inertia ixx="0.0001" ixy="0" ixz="0" iyy="0.0001" iyz="0" izz="0.0001"/>
+    </inertial>
+  </link>
+  <joint name="lidar_joint" type="fixed">
+    <parent link="base_link"/>
+    <child link="lidar_link"/>
+    <origin xyz="${body_length/2 - 0.03} 0 ${body_height/2 + 0.025}" rpy="0 0 0"/>
+  </joint>
+  <gazebo reference="lidar_link">
+    <sensor name="lidar_sensor" type="ray">
+      <always_on>true</always_on>
+      <update_rate>20.0</update_rate>
+      <visualize>true</visualize>
+      <ray>
+        <scan>
+          <horizontal>
+            <samples>720</samples>
+            <resolution>1</resolution>
+            <min_angle>-1.5708</min_angle>
+            <max_angle>1.5708</max_angle>
+          </horizontal>
+        </scan>
+        <range>
+          <min>0.1</min>
+          <max>12.0</max>
+          <resolution>0.01</resolution>
+        </range>
+        <noise>
+          <type>gaussian</type>
+          <mean>0.0</mean>
+          <stddev>0.01</stddev>
+        </noise>
+      </ray>
+      <plugin name="gazebo_ros_laser" filename="libgazebo_ros_ray_sensor.so">
+        <topicName>scan</topicName>
+        <frameName>lidar_link</frameName>
+      </plugin>
+    </sensor>
+  </gazebo>
   <!-- Makro koła -->
   <xacro:macro name="wheel" params="side wheel_side_sign joint_sign index x_offset">
@@ -113,4 +214,10 @@
     <material>Gazebo/Grey</material>
   </gazebo>
+  <gazebo reference="depth_camera_link">
+    <material>Gazebo/Black</material>
+  </gazebo>
+  <gazebo reference="lidar_link">
+    <material>Gazebo/Black</material>
+  </gazebo>
   <!-- Plugin ros2_control -->
   <gazebo>

Commit message: merge scripts

File: src/boxygo/urdf/6_wheel_robot_v2.urdf.xacro (robot description, xacro)
@@ -34,15 +34,19 @@
   </link>
     <!-- Kamera -->
+  <joint name="depth_camera_joint" type="fixed">
+    <parent link="base_link"/>
+    <child link="depth_camera_link"/>
+    <origin xyz="${body_length/2 + 0.01} 0 0.1" rpy="0 0 0"/>
+  </joint>
   <link name="depth_camera_link">
     <visual>
       <geometry>
-        <box size="0.05 0.05 0.05"/>
-      </geometry>
-      <origin xyz="0 0 0" rpy="0 0 0"/>
+        <box size="0.02 0.09 0.03"/>
+      </geometry>
       <material name="black"/>
     </visual>
     <collision>
       <geometry>
-        <box size="0.05 0.05 0.05"/>
+        <box size="0.02 0.09 0.03"/>
       </geometry>
     </collision>
@@ -52,29 +56,31 @@
     </inertial>
   </link>
-  <joint name="depth_camera_joint" type="fixed">
-    <parent link="base_link"/>
-    <child link="depth_camera_link"/>
-    <origin xyz="${body_length/2 + 0.025} 0 ${body_height/2 - 0.025 - 0.05}" rpy="0 0 0"/>
+  <joint name="depth_camera_optical_joint" type="fixed">
+    <parent link="depth_camera_link"/>
+    <child link="depth_camera_link_optical"/>
+    <origin xyz="0 0 0" rpy="${-pi/2} 0 ${-pi/2}"/> <!-- Standard ROS transform: optical frame (Z forward, X right, Y down) -->
   </joint>
+  <link name="depth_camera_link_optical"></link>
   <gazebo reference="depth_camera_link">
-    <sensor name="depth_camera_sensor" type="camera">
-      <always_on>true</always_on>
+    <sensor name="depth_camera" type="depth">
+      <pose> 0 0 0 0 0 0 </pose>
       <visualize>true</visualize>
-      <update_rate>30.0</update_rate>
+      <update_rate>10</update_rate>
       <camera>
-        <horizontal_fov>1.39626</horizontal_fov>
+        <horizontal_fov>1.089</horizontal_fov>
         <image>
+          <format>B8G8R8</format>
           <width>640</width>
           <height>480</height>
-          <format>R8G8B8</format>
         </image>
         <clip>
-          <near>0.1</near>
-          <far>10.0</far>
+          <near>0.05</near>
+          <far>8.0</far>
         </clip>
       </camera>
       <plugin name="depth_camera_controller" filename="libgazebo_ros_camera.so">
-        <camera_name>depth_camera</camera_name>
-        <frame_name>depth_camera_link</frame_name>
+        <frame_name>depth_camera_link_optical</frame_name>
+        <min_depth>0.1</min_depth>
+        <max_depth>100.0</max_depth>
       </plugin>
     </sensor>
