Commit message: add maping

File: src/boxygo/urdf/6_wheel_robot.urdf.xacro (robot description, xacro)
@@ -34,103 +34,117 @@
     </inertial>
   </link>
-  <!-- Makro koła -->
-  <xacro:macro name="wheel" params="side parent_link wheel_side_sign joint_sign index x_offset">
-    <xacro:property name="ixx" value="${(1.0/12.0) * wheel_mass * (3 * wheel_radius**2 + wheel_width**2)}"/>
-    <xacro:property name="izz" value="${0.5 * wheel_mass * wheel_radius**2}"/>
-    <link name="${side}_wheel_${index}">
-      <inertial>
-        <mass value="${wheel_mass}"/>
-        <inertia ixx="${ixx}" iyy="${ixx}" izz="${izz}" ixy="0.0" ixz="0.0" iyz="0.0"/>
-      </inertial>
-      <visual>
-        <geometry>
-          <mesh filename="${pkg_path}/meshes/hov_wheel_short_look.stl" scale="0.001 0.001 0.001"/>
-        </geometry>
-        <origin xyz="0 0 0" rpy="0 0 ${wheel_side_sign * math.pi}"/>
-        <material name="grey"/>
-      </visual>
-      <collision>
-        <geometry>
-          <mesh filename="${pkg_path}/meshes/hov_wheel_short_colision.stl" scale="0.001 0.001 0.001"/>
-        </geometry>
-        <origin xyz="0 0 0" rpy="0 0 ${wheel_side_sign * math.pi}"/>
-      </collision>
+  <!-- footprint-->
+  <joint name="base_footprint_joint" type="fixed">
+        <parent link="base_link"/>
+        <child link="base_footprint"/>
+        <origin xyz="0 0 0" rpy="0 0 0"/>
+    </joint>
+    <link name="base_footprint">
     </link>
-    <gazebo reference="${side}_wheel_${index}">
-      <mu1>1.0</mu1>
-      <mu2>1.0</mu2>
-      <kp>100000.0</kp>
-      <kd>10.0</kd>
-      <minDepth>0.001</minDepth>
-      <maxVel>0.01</maxVel>
-    </gazebo>
-    <joint name="${side}_wheel_${index}_joint" type="continuous">
-      <parent link="${parent_link}"/>
-      <child link="${side}_wheel_${index}"/>
-      <origin xyz="${x_offset} ${joint_sign * wheel_y_offset} ${z_offset}" rpy="0 0 0"/>
-      <axis xyz="0 1 0"/>
-      <limit effort="10.0" velocity="10.0"/>
-      <dynamics damping="0.1" friction="0.1"/>
-    </joint>
-    <transmission name="${side}_wheel_${index}_trans">
-    <type>transmission_interface/SimpleTransmission</type>
-    <joint name="${side}_wheel_${index}_joint">
-      <hardwareInterface>hardware_interface/VelocityJointInterface</hardwareInterface>
-    </joint>
-    <actuator name="${side}_wheel_${index}_motor">
-      <hardwareInterface>hardware_interface/VelocityJointInterface</hardwareInterface>
-      <mechanicalReduction>1</mechanicalReduction>
-    </actuator>
-  </transmission>
-  </xacro:macro>
-  <xacro:macro name="wheel_beam" params="side beam_link wheel_side_sign index x_offset y_offset">
-    <xacro:property name="ixx" value="${(1.0/12.0) * wheel_mass * (3 * wheel_radius**2 + wheel_width**2)}"/>
-    <xacro:property name="izz" value="${0.5 * wheel_mass * wheel_radius**2}"/>
-    <link name="${side}_wheel_${index}">
-      <inertial>
-        <mass value="${wheel_mass}"/>
-        <inertia ixx="${ixx}" iyy="${ixx}" izz="${izz}" ixy="0.0" ixz="0.0" iyz="0.0"/>
-      </inertial>
-      <visual>
-        <geometry>
-          <mesh filename="${pkg_path}/meshes/hov_wheel_short_look.stl" scale="0.001 0.001 0.001"/>
-        </geometry>
-        <origin xyz="0 0 0" rpy="0 0 ${wheel_side_sign * math.pi}"/>
-        <material name="grey"/>
-      </visual>
-      <collision>
-        <geometry>
-          <mesh filename="${pkg_path}/meshes/hov_wheel_short_colision.stl" scale="0.001 0.001 0.001"/>
-        </geometry>
-        <origin xyz="0 0 0" rpy="0 0 ${wheel_side_sign * math.pi}"/>
-      </collision>
-    </link>
-    <gazebo reference="${side}_wheel_${index}">
-      <mu1>1.0</mu1>
-      <mu2>1.0</mu2>
-      <kp>100000.0</kp>
-      <kd>10.0</kd>
-      <minDepth>0.001</minDepth>
-      <maxVel>0.01</maxVel>
-    </gazebo>
-    <joint name="${side}_wheel_${index}_joint" type="continuous">
-      <parent link="${beam_link}"/>
-      <child link="${side}_wheel_${index}"/>
-      <origin xyz="${x_offset} ${y_offset} 0" rpy="0 0 0"/>
-      <axis xyz="0 1 0"/>
-      <limit effort="10.0" velocity="10.0"/>
-      <dynamics damping="0.1" friction="0.1"/>
-    </joint>
-    <transmission name="${side}_wheel_${index}_trans">
-      <type>transmission_interface/SimpleTransmission</type>
-      <joint name="${side}_wheel_${index}_joint">
-        <hardwareInterface>hardware_interface/VelocityJointInterface</hardwareInterface>
-      </joint>
-      <actuator name="${side}_wheel_${index}_motor">
-        <hardwareInterface>hardware_interface/VelocityJointInterface</hardwareInterface>
-        <mechanicalReduction>1</mechanicalReduction>
-      </actuator>
-    </transmission>
-  </xacro:macro>
+    <!-- Kamera -->
+  <link name="depth_camera_link">
+    <visual>
+      <geometry>
+        <box size="0.05 0.05 0.05"/>
+      </geometry>
+      <origin xyz="0 0 0" rpy="0 0 0"/>
+      <material name="black"/>
+    </visual>
+    <collision>
+      <geometry>
+        <box size="0.05 0.05 0.05"/>
+      </geometry>
+    </collision>
+    <inertial>
+      <mass value="0.1"/>
+      <inertia ixx="0.0001" ixy="0.0" ixz="0.0" iyy="0.0001" iyz="0.0" izz="0.0001"/>
+    </inertial>
+  </link>
+  <joint name="depth_camera_joint" type="fixed">
+    <parent link="base_link"/>
+    <child link="depth_camera_link"/>
+    <origin xyz="${body_length/2 + 0.025} 0 ${body_height/2 - 0.025 - 0.05}" rpy="0 0 0"/>
+  </joint>
+  <gazebo reference="depth_camera_link">
+    <sensor name="depth_camera_sensor" type="camera">
+      <always_on>true</always_on>
+      <visualize>true</visualize>
+      <update_rate>30.0</update_rate>
+      <camera>
+        <horizontal_fov>1.39626</horizontal_fov>
+        <image>
+          <width>640</width>
+          <height>480</height>
+          <format>R8G8B8</format>
+        </image>
+        <clip>
+          <near>0.1</near>
+          <far>10.0</far>
+        </clip>
+      </camera>
+      <plugin name="depth_camera_controller" filename="libgazebo_ros_camera.so">
+        <camera_name>depth_camera</camera_name>
+        <frame_name>depth_camera_link</frame_name>
+      </plugin>
+    </sensor>
+  </gazebo>
+    <!-- Lidar 2D -->
+  <link name="lidar_link">
+    <visual>
+      <geometry>
+        <cylinder length="0.05" radius="0.03"/>
+      </geometry>
+      <material name="black"/>
+    </visual>
+    <collision>
+      <geometry>
+        <cylinder length="0.05" radius="0.03"/>
+      </geometry>
+    </collision>
+    <inertial>
+      <mass value="0.2"/>
+      <inertia ixx="0.0001" ixy="0" ixz="0" iyy="0.0001" iyz="0" izz="0.0001"/>
+    </inertial>
+  </link>
+  <joint name="lidar_joint" type="fixed">
+    <parent link="base_link"/>
+    <child link="lidar_link"/>
+    <origin xyz="${body_length/2 - 0.03} 0 ${body_height/2 + 0.025}" rpy="0 0 0"/>
+  </joint>
+  <gazebo reference="lidar_link">
+    <sensor name="lidar_sensor" type="ray">
+      <always_on>true</always_on>
+      <update_rate>10.0</update_rate>
+      <visualize>true</visualize>
+      <ray>
+        <scan>
+          <horizontal>
+            <samples>360</samples>
+            <resolution>1</resolution>
+            <min_angle>-3.14159</min_angle>
+            <max_angle>3.14159</max_angle>
+          </horizontal>
+        </scan>
+        <range>
+          <min>0.3</min>
+          <max>12</max>
+          <resolution>0.01</resolution>
+        </range>
+        <noise>
+          <type>gaussian</type>
+          <mean>0.0</mean>
+          <stddev>0.01</stddev>
+        </noise>
+      </ray>
+      <plugin name="gazebo_ros_laser" filename="libgazebo_ros_ray_sensor.so">
+        <topicName>scan</topicName>
+        <ros>
+            <argument>~/out:=scan</argument>
+        </ros>
+        <output_type>sensor_msgs/LaserScan</output_type>
+        <frameName>lidar_link</frameName>
+      </plugin>
+    </sensor>
+  </gazebo>
   <link name="left_rocker_beam">
     <inertial>
@@ -314,4 +328,10 @@
     <material>Gazebo/Grey</material>
   </gazebo>
+  <gazebo reference="depth_camera_link">
+    <material>Gazebo/Black</material>
+  </gazebo>
+  <gazebo reference="lidar_link">
+    <material>Gazebo/Black</material>
+  </gazebo>
   <!-- Plugin ros2_control -->
   <gazebo>

Commit message: IMU sensor

File: src/boxygo/urdf/6_wheel_robot.urdf.xacro (robot description, xacro)
@@ -34,4 +34,44 @@
     </inertial>
   </link>
+  <!-- IMU sensor -->
+  <link name="imu_link">
+    <inertial>
+      <mass value="0.01"/>
+      <origin xyz="0 0 0" rpy="0 0 0"/>
+      <inertia ixx="1e-5" ixy="0" ixz="0" iyy="1e-5" iyz="0" izz="1e-5"/>
+    </inertial>
+  </link>
+  <joint name="imu_joint" type="fixed">
+    <parent link="base_link"/>
+    <child link="imu_link"/>
+    <origin xyz="0 0 ${body_height/2}" rpy="0 0 0"/>
+  </joint>
+  <gazebo reference="imu_link">
+    <sensor type="imu" name="imu_sensor">
+      <always_on>true</always_on>
+      <update_rate>2.0</update_rate>
+      <imu>
+        <noise>
+          <angular_velocity>
+            <type>gaussian</type>
+            <mean>0.0</mean>
+            <stddev>0.001</stddev>
+          </angular_velocity>
+          <linear_acceleration>
+            <type>gaussian</type>
+            <mean>0.0</mean>
+            <stddev>0.001</stddev>
+          </linear_acceleration>
+        </noise>
+      </imu>
+      <plugin name="imu_plugin" filename="libgazebo_ros_imu_sensor.so">
+        <ros>
+          <namespace>/</namespace>
+          <remapping>~/out:=imu/data</remapping>
+        </ros>
+        <frame_name>imu_link</frame_name>
+      </plugin>
+    </sensor>
+  </gazebo>
   <!-- footprint-->
   <joint name="base_footprint_joint" type="fixed">
@@ -231,10 +271,10 @@
   </link>
   <gazebo reference="${side}_wheel_${index}">
-    <mu1>1.0</mu1>
-    <mu2>1.0</mu2>
+    <mu1>5.0</mu1>
+    <mu2>5.0</mu2>
     <kp>100000.0</kp>
     <kd>10.0</kd>
     <minDepth>0.001</minDepth>
-    <maxVel>0.01</maxVel>
+    <maxVel>0.1</maxVel>
   </gazebo>
   <joint name="${side}_wheel_${index}_joint" type="continuous">

Commit message: add tf

File: src/boxygo/urdf/6_wheel_robot.urdf.xacro (robot description, xacro)
@@ -423,4 +423,14 @@
       <state_interface name="velocity"/>
     </joint>
+    <joint name="left_rocker_beam_joint">
+      <command_interface name="position"/>
+      <state_interface name="position"/>
+      <state_interface name="velocity"/>
+    </joint>
+    <joint name="right_rocker_beam_joint">
+      <command_interface name="position"/>
+      <state_interface name="position"/>
+      <state_interface name="velocity"/>
+    </joint>
   </ros2_control>
 </robot>

Commit message: meshes update, sensors fusion update

File: src/boxygo/urdf/6_wheel_robot.urdf.xacro (robot description, xacro)
@@ -50,5 +50,5 @@
     <sensor type="imu" name="imu_sensor">
       <always_on>true</always_on>
-      <update_rate>2.0</update_rate>
+      <update_rate>60.0</update_rate>
       <imu>
         <noise>
@@ -71,4 +71,7 @@
         </ros>
         <frame_name>imu_link</frame_name>
+        <orientation>0.01 0 0  0 0.01 0  0 0 0.01</orientation>
+        <angular_velocity>0.01 0 0  0 0.01 0  0 0 0.01</angular_velocity>
+        <linear_acceleration>999 0 0  0 999 0  0 0 999</linear_acceleration>
       </plugin>
     </sensor>
@@ -115,5 +118,5 @@
       <pose>0 0 0 0 0 0</pose>
       <visualize>true</visualize>
-      <update_rate>30.0</update_rate>
+      <update_rate>60.0</update_rate>
       <camera>
         <horizontal_fov>1.39626</horizontal_fov>
@@ -162,5 +165,5 @@
     <sensor name="lidar_sensor" type="ray">
       <always_on>true</always_on>
-      <update_rate>10.0</update_rate>
+      <update_rate>60.0</update_rate>
       <visualize>true</visualize>
       <ray>
@@ -201,5 +204,5 @@
     <visual>
       <geometry>
-        <mesh filename="${pkg_path}/meshes/rocker_model.stl" scale="0.001 0.001 0.001"/>
+        <mesh filename="file://${pkg_path}/meshes/rocker_model.stl" scale="0.001 0.001 0.001"/>
       </geometry>
       <origin xyz="0 0 0" rpy="0 0 0"/>
@@ -208,5 +211,5 @@
     <collision>
       <geometry>
-        <mesh filename="${pkg_path}/meshes/rocker_model.stl" scale="0.001 0.001 0.001"/>
+        <mesh filename="file://${pkg_path}/meshes/rocker_model.stl" scale="0.001 0.001 0.001"/>
       </geometry>
       <origin xyz="0 0 0" rpy="0 0 0"/>
@@ -228,5 +231,5 @@
   <visual>
     <geometry>
-      <mesh filename="${pkg_path}/meshes/rocker_model.stl" scale="0.001 0.001 0.001"/>
+      <mesh filename="file://${pkg_path}/meshes/rocker_model.stl" scale="0.001 0.001 0.001"/>
     </geometry>
     <origin xyz="0 0 0" rpy="0 0 ${math.pi}"/>
@@ -235,5 +238,5 @@
   <collision>
     <geometry>
-      <mesh filename="${pkg_path}/meshes/rocker_model.stl" scale="0.001 0.001 0.001"/>
+      <mesh filename="file://${pkg_path}/meshes/rocker_model.stl" scale="0.001 0.001 0.001"/>
     </geometry>
     <origin xyz="0 0 0" rpy="0 0 ${math.pi}"/>
@@ -258,5 +261,5 @@
     <visual>
       <geometry>
-        <mesh filename="${pkg_path}/meshes/hov_wheel_short_look.stl" scale="0.001 0.001 0.001"/>
+        <mesh filename="file://${pkg_path}/meshes/hov_wheel_short_look.stl" scale="0.001 0.001 0.001"/>
       </geometry>
       <origin xyz="0 0 0" rpy="0 0 ${wheel_side_sign * math.pi}"/>
@@ -265,5 +268,5 @@
     <collision>
       <geometry>
-        <mesh filename="${pkg_path}/meshes/hov_wheel_short_colision.stl" scale="0.001 0.001 0.001"/>
+        <mesh filename="file://${pkg_path}/meshes/hov_wheel_short_look.stl" scale="0.001 0.001 0.001"/>
       </geometry>
       <origin xyz="0 0 0" rpy="0 0 ${wheel_side_sign * math.pi}"/>
@@ -384,5 +387,5 @@
   <gazebo>
     <plugin name="gazebo_ros2_control" filename="libgazebo_ros2_control.so">
-      <update_rate>30</update_rate>
+      <update_rate>60</update_rate>
       <parameters>${pkg_path}/config/diff_drive_controller_v1.yaml</parameters>
     </plugin>

Commit message: depth-camera - D 435imesh added to simulation in Gazebo

File: src/boxygo/urdf/6_wheel_robot.urdf.xacro (robot description, xacro)
@@ -1,4 +1,5 @@
 <?xml version="1.0"?>
 <robot name="delivery_robot" xmlns:xacro="http://ros.org/wiki/xacro">
+  <xacro:include filename="_d435i.urdf.xacro"/>
   <!-- Właściwości -->
   <xacro:property name="body_length" value="0.9"/>
@@ -34,55 +35,5 @@
     </inertial>
   </link>
-  <!-- IMU sensor -->
-  <link name="imu_link">
-    <inertial>
-      <mass value="0.01"/>
-      <origin xyz="0 0 0" rpy="0 0 0"/>
-      <inertia ixx="1e-5" ixy="0" ixz="0" iyy="1e-5" iyz="0" izz="1e-5"/>
-    </inertial>
-  </link>
-  <joint name="imu_joint" type="fixed">
-    <parent link="base_link"/>
-    <child link="imu_link"/>
-    <origin xyz="0 0 ${body_height/2}" rpy="0 0 0"/>
-  </joint>
-  <gazebo reference="imu_link">
-    <sensor type="imu" name="imu_sensor">
-      <always_on>true</always_on>
-      <update_rate>60.0</update_rate>
-      <imu>
-        <noise>
-          <angular_velocity>
-            <type>gaussian</type>
-            <mean>0.0</mean>
-            <stddev>0.001</stddev>
-          </angular_velocity>
-          <linear_acceleration>
-            <type>gaussian</type>
-            <mean>0.0</mean>
-            <stddev>0.001</stddev>
-          </linear_acceleration>
-        </noise>
-      </imu>
-      <plugin name="imu_plugin" filename="libgazebo_ros_imu_sensor.so">
-        <ros>
-          <namespace>/</namespace>
-          <remapping>~/out:=imu/data</remapping>
-        </ros>
-        <frame_name>imu_link</frame_name>
-        <orientation>0.01 0 0  0 0.01 0  0 0 0.01</orientation>
-        <angular_velocity>0.01 0 0  0 0.01 0  0 0 0.01</angular_velocity>
-        <linear_acceleration>999 0 0  0 999 0  0 0 999</linear_acceleration>
-      </plugin>
-    </sensor>
-  </gazebo>
-  <!-- footprint-->
-  <joint name="base_footprint_joint" type="fixed">
-        <parent link="base_link"/>
-        <child link="base_footprint"/>
-        <origin xyz="0 0 0" rpy="0 0 0"/>
-    </joint>
-    <link name="base_footprint">
-    </link>
+<<<<<<< Updated upstream
     <!-- Kamera -->
   <link name="depth_camera_link">
@@ -139,4 +90,6 @@
     </sensor>
   </gazebo>
+=======
+>>>>>>> Stashed changes
     <!-- Lidar 2D -->
   <link name="lidar_link">
@@ -197,4 +150,8 @@
     </sensor>
   </gazebo>
+  <!-- Kamera D435i -->
+  <xacro:sensor_d435i parent="base_link" name="camera" topics_ns="camera">
+        <origin xyz="${body_length/2 + 0.01} 0 ${body_height/2 - 0.1}" rpy="0.0 0.0 0.0"/>
+  </xacro:sensor_d435i>
   <link name="left_rocker_beam">
     <inertial>
@@ -381,7 +338,4 @@
     <material>Gazebo/Black</material>
   </gazebo>
-  <gazebo reference="depth_camera_link">
-    <material>Gazebo/Black</material>
-  </gazebo>
   <!-- Plugin ros2_control -->
   <gazebo>
