Commit message: fix wheel

File: src/boxygo/urdf/robot_luksusowy.urdf.xacro (robot description, xacro)
@@ -130,5 +130,5 @@
       <visual>
         <geometry>
-          <mesh filename="file://${pkg_path}/meshes/wheel.stl" scale="0.001 0.001 0.001"/>
+          <mesh filename="file://${pkg_path}/meshes/wheel.dae" scale="0.001 0.001 0.001"/>
         </geometry>
         <origin xyz="0 0 0" rpy="0 0 0"/>
@@ -137,5 +137,5 @@
       <collision>
         <geometry>
-          <mesh filename="file://${pkg_path}/meshes/wheel.stl" scale="0.001 0.001 0.001"/>
+          <mesh filename="file://${pkg_path}/meshes/wheel.dae" scale="0.001 0.001 0.001"/>
         </geometry>
         <origin xyz="0 0 0" rpy="0 0 0"/>
