Commit message: add our robot to issac sim and configure setup for lidar

File: src/boxygo_description/urdf/robot_luksusowy.urdf.xacro (robot description, xacro)
@@ -26,6 +26,6 @@
   <xacro:include filename="$(find boxygo_description)/urdf/sensors.urdf.xacro"/>
   <xacro:add_sensors parent="base_link"
-                    body_length="${body_length}"
-                    body_height="${body_height}"/>
+                     body_length="${body_length}"
+                     body_height="${body_height}"/>
   <!-- Rama -->
   <link name="base_link">
@@ -33,5 +33,5 @@
       <origin xyz="0 0 0" rpy="0 0 0"/>
       <geometry>
-        <mesh filename="file://${boxygo_description_pkg}/meshes/frame_full.stl" scale="0.001 0.001 0.001"/>
+        <mesh filename="meshes/frame_full.stl" scale="0.001 0.001 0.001"/>
       </geometry>
       <material name="darkgrey"/>
@@ -40,5 +40,5 @@
       <origin xyz="0 0 0" rpy="0 0 0"/>
       <geometry>
-        <mesh filename="file://${boxygo_description_pkg}/meshes/frame_full.stl" scale="0.001 0.001 0.001"/>
+        <mesh filename="meshes/frame_full.stl" scale="0.001 0.001 0.001"/>
       </geometry>
     </collision>
@@ -49,33 +49,9 @@
     </inertial>
   </link>
-  <!-- Korpus -->
-  <!-- <link name="body_link">
-    <visual>
-      <geometry>
-        <box size="${body_length} ${body_width} ${body_height}"/>
-      </geometry>
-      <material name="white"/>
-    </visual>
-    <collision>
-      <geometry>
-        <box size="${body_length} ${body_width} ${body_height}"/>
-      </geometry>
-    </collision>
-    <inertial>
-      <mass value="${body_mass}"/>
-      <origin xyz="0 0 0" rpy="0 0 0"/>
-      <inertia ixx="0.50108" iyy="0.75508" izz="0.83949" ixy="0" ixz="0" iyz="0"/>
-    </inertial>
-  </link>
-  <joint name="body_link_joint" type="fixed">
-    <parent link="base_link"/>
-    <child link="body_link"/>
-    <origin xyz="${body_x_offset} 0 ${body_height/2 + 0.1752}" rpy="0 0 0"/>
-  </joint> -->
   <!-- Belki -->
   <link name="right_rocker_beam">
     <visual>
       <geometry>
-        <mesh filename="file://${boxygo_description_pkg}/meshes/beam_full.stl" scale="0.001 0.001 0.001"/>
+        <mesh filename="meshes/beam_full.stl" scale="0.001 0.001 0.001"/>
       </geometry>
       <origin xyz="0 0 0" rpy="0 0 0"/>
@@ -84,5 +60,5 @@
     <collision>
       <geometry>
-        <mesh filename="file://${boxygo_description_pkg}/meshes/beam_full.stl" scale="0.001 0.001 0.001"/>
+        <mesh filename="meshes/beam_full.stl" scale="0.001 0.001 0.001"/>
       </geometry>
       <origin xyz="0 0 0" rpy="0 0 0"/>
@@ -105,5 +81,5 @@
     <visual>
       <geometry>
-        <mesh filename="file://${boxygo_description_pkg}/meshes/beam_full.stl" scale="0.001 0.001 0.001"/>
+        <mesh filename="meshes/beam_full.stl" scale="0.001 0.001 0.001"/>
       </geometry>
       <origin xyz="0 0 0" rpy="0 0 0"/>
@@ -112,5 +88,5 @@
     <collision>
       <geometry>
-        <mesh filename="file://${boxygo_description_pkg}/meshes/beam_full.stl" scale="0.001 0.001 0.001"/>
+        <mesh filename="meshes/beam_full.stl" scale="0.001 0.001 0.001"/>
       </geometry>
       <origin xyz="0 0 0" rpy="0 0 0"/>
@@ -135,5 +111,5 @@
       <visual>
         <geometry>
-          <mesh filename="file://${boxygo_description_pkg}/meshes/wheel.dae" scale="0.001 0.001 0.001"/>
+          <mesh filename="meshes/wheel.dae" scale="0.001 0.001 0.001"/>
         </geometry>
         <origin xyz="0 0 0" rpy="0 0 0"/>
@@ -142,5 +118,5 @@
       <collision>
         <geometry>
-          <mesh filename="file://${boxygo_description_pkg}/meshes/wheel.dae" scale="0.001 0.001 0.001"/>
+          <mesh filename="meshes/wheel.dae" scale="0.001 0.001 0.001"/>
         </geometry>
         <origin xyz="0 0 0" rpy="0 0 0"/>

Commit message: hardware interface implemented

File: src/boxygo_description/urdf/robot_luksusowy.urdf.xacro (robot description, xacro)
@@ -197,5 +197,66 @@
     </plugin>
   </gazebo>
-  <!-- ros2_control hardware -->
+  <ros2_control name="BoxygoMoteusSystem" type="system">
+  <hardware>
+    <plugin>moteus_hardware_interface/MoteusHardwareInterface</plugin>
+  </hardware>
+  <!-- Koła lewe -->
+  <joint name="left_wheel_1_joint">
+    <param name="can_protocol">moteus</param>
+    <param name="can_id">1</param>
+    <param name="axis_direction">-1</param>
+    <param name="gear_ratio">1.0</param>
+    <command_interface name="velocity"/>
+    <state_interface name="position"/>
+    <state_interface name="velocity"/>
+  </joint>
+  <joint name="left_wheel_2_joint">
+    <param name="can_protocol">moteus</param>
+    <param name="can_id">2</param>
+    <param name="axis_direction">-1</param>
+    <param name="gear_ratio">1.0</param>
+    <command_interface name="velocity"/>
+    <state_interface name="position"/>
+    <state_interface name="velocity"/>
+  </joint>
+  <joint name="left_wheel_3_joint">
+    <param name="can_protocol">moteus</param>
+    <param name="can_id">3</param>
+    <param name="axis_direction">-1</param>
+    <param name="gear_ratio">1.0</param>
+    <command_interface name="velocity"/>
+    <state_interface name="position"/>
+    <state_interface name="velocity"/>
+  </joint>
+  <!-- Koła prawe -->
+  <joint name="right_wheel_1_joint">
+    <param name="can_protocol">moteus</param>
+    <param name="can_id">4</param>
+    <param name="axis_direction">1</param>
+    <param name="gear_ratio">1.0</param>
+    <command_interface name="velocity"/>
+    <state_interface name="position"/>
+    <state_interface name="velocity"/>
+  </joint>
+  <joint name="right_wheel_2_joint">
+    <param name="can_protocol">moteus</param>
+    <param name="can_id">5</param>
+    <param name="axis_direction">1</param>
+    <param name="gear_ratio">1.0</param>
+    <command_interface name="velocity"/>
+    <state_interface name="position"/>
+    <state_interface name="velocity"/>
+  </joint>
+  <joint name="right_wheel_3_joint">
+   <param name="can_protocol">moteus</param>
+    <param name="can_id">6</param>
+    <param name="axis_direction">1</param>
+    <param name="gear_ratio">1.0</param>
+    <command_interface name="velocity"/>
+    <state_interface name="position"/>
+    <state_interface name="velocity"/>
+  </joint>
+ </ros2_control>
+ <!-- ros2_control simulation
   <ros2_control name="BoxyGoSystem" type="system">
     <hardware>
@@ -242,4 +303,4 @@
       <state_interface name="velocity"/>
     </joint>
-  </ros2_control>
+  </ros2_control> -->
 </robot>

Commit message: update

File: src/boxygo_description/urdf/robot_luksusowy.urdf.xacro (robot description, xacro)
@@ -33,5 +33,5 @@
       <origin xyz="0 0 0" rpy="0 0 0"/>
       <geometry>
-        <mesh filename="meshes/frame_full.stl" scale="0.001 0.001 0.001"/>
+        <mesh filename="file://${boxygo_description_pkg}/meshes/frame_full.stl" scale="0.001 0.001 0.001"/>
       </geometry>
       <material name="darkgrey"/>
@@ -40,5 +40,5 @@
       <origin xyz="0 0 0" rpy="0 0 0"/>
       <geometry>
-        <mesh filename="meshes/frame_full.stl" scale="0.001 0.001 0.001"/>
+        <mesh filename="file://${boxygo_description_pkg}/meshes/frame_full.stl" scale="0.001 0.001 0.001"/>
       </geometry>
     </collision>
@@ -53,5 +53,5 @@
     <visual>
       <geometry>
-        <mesh filename="meshes/beam_full.stl" scale="0.001 0.001 0.001"/>
+        <mesh filename="file://${boxygo_description_pkg}/meshes/beam_full.stl" scale="0.001 0.001 0.001"/>
       </geometry>
       <origin xyz="0 0 0" rpy="0 0 0"/>
@@ -60,5 +60,5 @@
     <collision>
       <geometry>
-        <mesh filename="meshes/beam_full.stl" scale="0.001 0.001 0.001"/>
+        <mesh filename="file://${boxygo_description_pkg}/meshes/beam_full.stl" scale="0.001 0.001 0.001"/>
       </geometry>
       <origin xyz="0 0 0" rpy="0 0 0"/>
@@ -81,5 +81,5 @@
     <visual>
       <geometry>
-        <mesh filename="meshes/beam_full.stl" scale="0.001 0.001 0.001"/>
+        <mesh filename="file://${boxygo_description_pkg}/meshes/beam_full.stl" scale="0.001 0.001 0.001"/>
       </geometry>
       <origin xyz="0 0 0" rpy="0 0 0"/>
@@ -88,5 +88,5 @@
     <collision>
       <geometry>
-        <mesh filename="meshes/beam_full.stl" scale="0.001 0.001 0.001"/>
+        <mesh filename="file://${boxygo_description_pkg}/meshes/beam_full.stl" scale="0.001 0.001 0.001"/>
       </geometry>
       <origin xyz="0 0 0" rpy="0 0 0"/>
@@ -111,5 +111,5 @@
       <visual>
         <geometry>
-          <mesh filename="meshes/wheel.dae" scale="0.001 0.001 0.001"/>
+          <mesh filename="file://${boxygo_description_pkg}/meshes/wheel.dae" scale="0.001 0.001 0.001"/>
         </geometry>
         <origin xyz="0 0 0" rpy="0 0 0"/>
@@ -118,5 +118,5 @@
       <collision>
         <geometry>
-          <mesh filename="meshes/wheel.dae" scale="0.001 0.001 0.001"/>
+          <mesh filename="file://${boxygo_description_pkg}/meshes/wheel.dae" scale="0.001 0.001 0.001"/>
         </geometry>
         <origin xyz="0 0 0" rpy="0 0 0"/>
