Commit message: -add urdf generation script

File: src/boxygo_description/urdf/luksusowy_isaac.urdf (robot description, URDF)
Before this commit: robot delivery_robot, 10 links, 9 joints
Links:
- link base_link: geometry collision mesh filename=file:///workspaces/isaac_ros-dev/install/boxygo_description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 scale=0.001 0.001 0.001; visual mesh filename=file:///workspaces/isaac_ros-dev/install/boxygo_description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 scale=0.001 0.001 0.001
- link left_rocker_beam: geometry collision mesh filename=file:///workspaces/isaac_ros-dev/install/boxygo_description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 scale=0.001 0.001 0.001; visual mesh filename=file:///workspaces/isaac_ros-dev/install/boxygo_description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 scale=0.001 0.001 0.001
- link left_wheel_1: geometry collision mesh filename=file:///workspaces/isaac_ros-dev/install/boxygo_description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 scale=0.001 0.001 0.001; visual mesh filename=file:///workspaces/isaac_ros-dev/install/boxygo_description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 scale=0.001 0.001 0.001
- link left_wheel_2: geometry collision mesh filename=file:///workspaces/isaac_ros-dev/install/boxygo_description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 scale=0.001 0.001 0.001; visual mesh filename=file:///workspaces/isaac_ros-dev/install/boxygo_description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 scale=0.001 0.001 0.001
- link left_wheel_3: geometry collision mesh filename=file:///workspaces/isaac_ros-dev/install/boxygo_description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 scale=0.001 0.001 0.001; visual mesh filename=file:///workspaces/isaac_ros-dev/install/boxygo_description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 scale=0.001 0.001 0.001
- link right_rocker_beam: geometry collision mesh filename=file:///workspaces/isaac_ros-dev/install/boxygo_description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 scale=0.001 0.001 0.001; visual mesh filename=file:///workspaces/isaac_ros-dev/install/boxygo_description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 scale=0.001 0.001 0.001
- link right_wheel_1: geometry collision mesh filename=file:///workspaces/isaac_ros-dev/install/boxygo_description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 scale=0.001 0.001 0.001; visual mesh filename=file:///workspaces/isaac_ros-dev/install/boxygo_description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 scale=0.001 0.001 0.001
- link right_wheel_2: geometry collision mesh filename=file:///workspaces/isaac_ros-dev/install/boxygo_description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 scale=0.001 0.001 0.001; visual mesh filename=file:///workspaces/isaac_ros-dev/install/boxygo_description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 scale=0.001 0.001 0.001
- link right_wheel_3: geometry collision mesh filename=file:///workspaces/isaac_ros-dev/install/boxygo_description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 scale=0.001 0.001 0.001; visual mesh filename=file:///workspaces/isaac_ros-dev/install/boxygo_description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 scale=0.001 0.001 0.001
Joints:
- joint laser_joint: origin xyz=0.06 0.0 0.32 rpy=0 0 0 -> xyz=0.06 0.0 0.32 rpy=0 0 3.141592653589793
