Commit message: add camera urdf

File: src/boxygo_description/urdf/luksusowy.urdf.xacro (robot description, xacro)
@@ -14,4 +14,6 @@
   </xacro:if>
   <xacro:include filename="$(find boxygo_description)/urdf/common/lidar.xacro"/>
+  <xacro:include filename="$(find boxygo_description)/urdf/common/_d435i.urdf.xacro"/>
   <xacro:sensor_ydlidar parent_link="base_link" x_offset="0.06" y_offset="0.0" z_offset="0.32"/>
+  <xacro:sensor_d435i parent="base_link" use_nominal_extrinsics="true"> <origin xyz="0.38 0.0 0.225" rpy="0 0 0"/></xacro:sensor_d435i>
 </robot>

File: src/boxygo_description/urdf/luksusowy_isaac.urdf (robot description, URDF)
Before this commit: robot delivery_robot, 10 links, 9 joints
Links:
- added link camera_accel_frame
- added link camera_accel_optical_frame
- added link camera_bottom_screw_frame
- added link camera_color_frame
- added link camera_color_optical_frame
- added link camera_depth_frame
- added link camera_depth_optical_frame
- added link camera_gyro_frame
- added link camera_gyro_optical_frame
- added link camera_infra1_frame
- added link camera_infra1_optical_frame
- added link camera_infra2_frame
- added link camera_infra2_optical_frame
- added link camera_link, mass 0.072; collision box size=0.02505 0.09 0.025; visual mesh filename=package://realsense2_description/meshes/d435.dae
Joints:
- added joint camera_accel_joint: type fixed, parent camera_link, child camera_accel_frame, origin xyz=-0.01174 -0.00552 0.0051 rpy=0 0 0
- added joint camera_accel_optical_joint: type fixed, parent camera_accel_frame, child camera_accel_optical_frame, origin xyz=0 0 0 rpy=-1.5707963267948966 0 -1.5707963267948966
- added joint camera_color_joint: type fixed, parent camera_link, child camera_color_frame, origin xyz=0 0.015 0 rpy=0 0 0
- added joint camera_color_optical_joint: type fixed, parent camera_color_frame, child camera_color_optical_frame, origin xyz=0 0 0 rpy=-1.5707963267948966 0 -1.5707963267948966
- added joint camera_depth_joint: type fixed, parent camera_link, child camera_depth_frame, origin xyz=0 0 0 rpy=0 0 0
- added joint camera_depth_optical_joint: type fixed, parent camera_depth_frame, child camera_depth_optical_frame, origin xyz=0 0 0 rpy=-1.5707963267948966 0 -1.5707963267948966
- added joint camera_gyro_joint: type fixed, parent camera_link, child camera_gyro_frame, origin xyz=-0.01174 -0.00552 0.0051 rpy=0 0 0
- added joint camera_gyro_optical_joint: type fixed, parent camera_gyro_frame, child camera_gyro_optical_frame, origin xyz=0 0 0 rpy=-1.5707963267948966 0 -1.5707963267948966
- added joint camera_infra1_joint: type fixed, parent camera_link, child camera_infra1_frame, origin xyz=0 0.0 0 rpy=0 0 0
- added joint camera_infra1_optical_joint: type fixed, parent camera_infra1_frame, child camera_infra1_optical_frame, origin xyz=0 0 0 rpy=-1.5707963267948966 0 -1.5707963267948966
- added joint camera_infra2_joint: type fixed, parent camera_link, child camera_infra2_frame, origin xyz=0 -0.05 0 rpy=0 0 0
- added joint camera_infra2_optical_joint: type fixed, parent camera_infra2_frame, child camera_infra2_optical_frame, origin xyz=0 0 0 rpy=-1.5707963267948966 0 -1.5707963267948966
- added joint camera_joint: type fixed, parent base_link, child camera_bottom_screw_frame, origin xyz=0.38 0.0 0.225 rpy=0 0 0
- added joint camera_link_joint: type fixed, parent camera_bottom_screw_frame, child camera_link, origin xyz=0.010600000000000002 0.0175 0.0125 rpy=0 0 0
