Commit message: use_sim_time update

File: src/boxygo_description/urdf/common/robot_joints.xacro (robot description, xacro)
@@ -41,7 +41,7 @@
     x_offset="${wheel_front_x_offset}" y_offset="${wheel_front_y_offset}" z_offset="${wheel_front_z_offset}"/>
   <xacro:wheel_assembly side="left" parent_link="left_rocker_beam" sign="-1" wheel_side_sign="0" index="2"
+    x_offset="${-wheel_beam_x_offset}" y_offset="${wheel_beam_y_offset}" z_offset="${wheel_beam_z_offset}"/>
+  <xacro:wheel_assembly side="left" parent_link="left_rocker_beam" sign="-1" wheel_side_sign="0" index="3"
     x_offset="${wheel_beam_x_offset}" y_offset="${wheel_beam_y_offset}" z_offset="${wheel_beam_z_offset}"/>
-  <xacro:wheel_assembly side="left" parent_link="left_rocker_beam" sign="-1" wheel_side_sign="0" index="3"
-    x_offset="${-wheel_beam_x_offset}" y_offset="${wheel_beam_y_offset}" z_offset="${wheel_beam_z_offset}"/>
   <xacro:wheel_assembly side="right" parent_link="base_link" sign="1" wheel_side_sign="0" index="1"
     x_offset="${wheel_front_x_offset}" y_offset="${-wheel_front_y_offset}" z_offset="${wheel_front_z_offset}"/>

File: src/boxygo_description/urdf/luksusowy_isaac.urdf (robot description, URDF)
Before this commit: robot delivery_robot, 24 links, 23 joints
Joints:
- joint left_wheel_2_joint: origin xyz=0.13 -0.05415 -0.0982 rpy=0 0 0.0 -> xyz=-0.13 -0.05415 -0.0982 rpy=0 0 0.0
- joint left_wheel_3_joint: origin xyz=-0.13 -0.05415 -0.0982 rpy=0 0 0.0 -> xyz=0.13 -0.05415 -0.0982 rpy=0 0 0.0
