Commit message: add pad features, fix sim paths

File: src/boxygo_description/urdf/common/robot_core.xacro (robot description, xacro)
@@ -1,5 +1,5 @@
 <?xml version="1.0"?>
 <robot xmlns:xacro="http://ros.org/wiki/xacro">
-  <xacro:property name="boxygo_description_pkg" value="$(find boxygo_description)"/>
+  <!-- PARAMETRY -->
   <xacro:property name="body_length" value="0.81"/>
   <xacro:property name="body_width" value="0.5927"/>
@@ -17,13 +17,15 @@
   <xacro:property name="wheel_front_x_offset" value="${wheel_gap}"/>
   <xacro:property name="wheel_front_z_offset" value="-0.0106"/>
+  <!-- MATERIAŁY -->
   <material name="black"><color rgba="0.0 0.0 0.0 1.0"/></material>
   <material name="white"><color rgba="0.7 0.7 0.7 0.5"/></material>
   <material name="grey"><color rgba="0.4 0.4 0.4 1.0"/></material>
   <material name="darkgrey"><color rgba="0.05 0.05 0.05 1.0"/></material>
+  <!-- BASE LINK -->
   <link name="base_link">
     <visual>
       <origin xyz="0 0 0" rpy="0 0 0"/>
       <geometry>
-        <mesh filename="file://${boxygo_description_pkg}/meshes/frame_full.stl" scale="0.001 0.001 0.001"/>
+        <mesh filename="package://boxygo_description/meshes/frame_full.stl" scale="0.001 0.001 0.001"/>
       </geometry>
       <material name="darkgrey"/>
@@ -32,5 +34,5 @@
       <origin xyz="0 0 0" rpy="0 0 0"/>
       <geometry>
-        <mesh filename="file://${boxygo_description_pkg}/meshes/frame_full.stl" scale="0.001 0.001 0.001"/>
+        <mesh filename="package://boxygo_description/meshes/frame_full.stl" scale="0.001 0.001 0.001"/>
       </geometry>
     </collision>
@@ -41,8 +43,9 @@
     </inertial>
   </link>
+  <!-- RIGHT ROCKER BEAM -->
   <link name="right_rocker_beam">
     <visual>
       <geometry>
-        <mesh filename="file://${boxygo_description_pkg}/meshes/beam_full.stl" scale="0.001 0.001 0.001"/>
+        <mesh filename="package://boxygo_description/meshes/beam_full.stl" scale="0.001 0.001 0.001"/>
       </geometry>
       <origin xyz="0 0 0" rpy="0 0 0"/>
@@ -51,5 +54,5 @@
     <collision>
       <geometry>
-        <mesh filename="file://${boxygo_description_pkg}/meshes/beam_full.stl" scale="0.001 0.001 0.001"/>
+        <mesh filename="package://boxygo_description/meshes/beam_full.stl" scale="0.001 0.001 0.001"/>
       </geometry>
       <origin xyz="0 0 0" rpy="0 0 0"/>
@@ -61,8 +64,9 @@
     </inertial>
   </link>
+  <!-- LEFT ROCKER BEAM -->
   <link name="left_rocker_beam">
     <visual>
       <geometry>
-        <mesh filename="file://${boxygo_description_pkg}/meshes/beam_full.stl" scale="0.001 0.001 0.001"/>
+        <mesh filename="package://boxygo_description/meshes/beam_full.stl" scale="0.001 0.001 0.001"/>
       </geometry>
       <origin xyz="0 0 0" rpy="0 0 0"/>
@@ -71,5 +75,5 @@
     <collision>
       <geometry>
-        <mesh filename="file://${boxygo_description_pkg}/meshes/beam_full.stl" scale="0.001 0.001 0.001"/>
+        <mesh filename="package://boxygo_description/meshes/beam_full.stl" scale="0.001 0.001 0.001"/>
       </geometry>
       <origin xyz="0 0 0" rpy="0 0 0"/>
@@ -81,9 +85,10 @@
     </inertial>
   </link>
+  <!-- KOŁA -->
   <xacro:macro name="wheel_link" params="prefix index">
     <link name="${prefix}_wheel_${index}">
       <visual>
         <geometry>
-          <mesh filename="file://${boxygo_description_pkg}/meshes/wheel.dae" scale="0.001 0.001 0.001"/>
+          <mesh filename="package://boxygo_description/meshes/wheel.dae" scale="0.001 0.001 0.001"/>
         </geometry>
         <origin xyz="0 0 0" rpy="0 0 0"/>
@@ -92,5 +97,5 @@
       <collision>
         <geometry>
-          <mesh filename="file://${boxygo_description_pkg}/meshes/wheel.dae" scale="0.001 0.001 0.001"/>
+          <mesh filename="package://boxygo_description/meshes/wheel.dae" scale="0.001 0.001 0.001"/>
         </geometry>
         <origin xyz="0 0 0" rpy="0 0 0"/>

File: src/boxygo_description/urdf/luksusowy_isaac.urdf (robot description, URDF)
Before this commit: robot delivery_robot, 10 links, 9 joints
Links:
- link base_link: geometry collision mesh filename=package://boxygo_description/meshes/frame_full.stl scale=0.001 0.001 0.001; visual mesh filename=package://boxygo_description/meshes/frame_full.stl scale=0.001 0.001 0.001
- link left_rocker_beam: geometry collision mesh filename=package://boxygo_description/meshes/beam_full.stl scale=0.001 0.001 0.001; visual mesh filename=package://boxygo_description/meshes/beam_full.stl scale=0.001 0.001 0.001
- link left_wheel_1: geometry collision mesh filename=package://boxygo_description/meshes/wheel.dae scale=0.001 0.001 0.001; visual mesh filename=package://boxygo_description/meshes/wheel.dae scale=0.001 0.001 0.001
- link left_wheel_2: geometry collision mesh filename=package://boxygo_description/meshes/wheel.dae scale=0.001 0.001 0.001; visual mesh filename=package://boxygo_description/meshes/wheel.dae scale=0.001 0.001 0.001
- link left_wheel_3: geometry collision mesh filename=package://boxygo_description/meshes/wheel.dae scale=0.001 0.001 0.001; visual mesh filename=package://boxygo_description/meshes/wheel.dae scale=0.001 0.001 0.001
- link right_rocker_beam: geometry collision mesh filename=package://boxygo_description/meshes/beam_full.stl scale=0.001 0.001 0.001; visual mesh filename=package://boxygo_description/meshes/beam_full.stl scale=0.001 0.001 0.001
- link right_wheel_1: geometry collision mesh filename=package://boxygo_description/meshes/wheel.dae scale=0.001 0.001 0.001; visual mesh filename=package://boxygo_description/meshes/wheel.dae scale=0.001 0.001 0.001
- link right_wheel_2: geometry collision mesh filename=package://boxygo_description/meshes/wheel.dae scale=0.001 0.001 0.001; visual mesh filename=package://boxygo_description/meshes/wheel.dae scale=0.001 0.001 0.001
- link right_wheel_3: geometry collision mesh filename=package://boxygo_description/meshes/wheel.dae scale=0.001 0.001 0.001; visual mesh filename=package://boxygo_description/meshes/wheel.dae scale=0.001 0.001 0.001

Commit message: fix isaac sim, restructurize launch

File: src/boxygo_description/urdf/common/robot_core.xacro (robot description, xacro)
@@ -90,5 +90,5 @@
       <visual>
         <geometry>
-          <mesh filename="package://boxygo_description/meshes/wheel.dae" scale="0.001 0.001 0.001"/>
+          <mesh filename="package://boxygo_description/meshes/wheel.stl" scale="0.001 0.001 0.001"/>
         </geometry>
         <origin xyz="0 0 0" rpy="0 0 0"/>

File: src/boxygo_description/urdf/config/isaac.xacro (robot description, xacro)
@@ -7,4 +7,7 @@
       <param name="joint_states_topic">/isaac_joint_states</param>
       <param name="sum_wrapped_joint_states">true</param>
+      <param name="provide_odom_frame">false</param>
+      <param name="publish_odom">false</param>
+      <param name="publish_odom_tf">false</param>
     </hardware>
     <joint name="left_wheel_1_joint">
@@ -38,4 +41,14 @@
       <state_interface name="velocity"/>
     </joint>
+    <joint name="left_rocker_beam_joint">
+      <command_interface name="velocity"/>
+      <state_interface name="position"/>
+      <state_interface name="velocity"/>
+    </joint>
+    <joint name="right_rocker_beam_joint">
+      <command_interface name="velocity"/>
+      <state_interface name="position"/>
+      <state_interface name="velocity"/>
+    </joint>
   </ros2_control>
 </robot>

File: src/boxygo_description/urdf/luksusowy_isaac.urdf (robot description, URDF)
Before this commit: robot delivery_robot, 24 links, 23 joints
Links:
- link left_wheel_1: geometry collision mesh filename=package://boxygo_description/meshes/wheel.dae scale=0.001 0.001 0.001; visual mesh filename=package://boxygo_description/meshes/wheel.stl scale=0.001 0.001 0.001
- link left_wheel_2: geometry collision mesh filename=package://boxygo_description/meshes/wheel.dae scale=0.001 0.001 0.001; visual mesh filename=package://boxygo_description/meshes/wheel.stl scale=0.001 0.001 0.001
- link left_wheel_3: geometry collision mesh filename=package://boxygo_description/meshes/wheel.dae scale=0.001 0.001 0.001; visual mesh filename=package://boxygo_description/meshes/wheel.stl scale=0.001 0.001 0.001
- link right_wheel_1: geometry collision mesh filename=package://boxygo_description/meshes/wheel.dae scale=0.001 0.001 0.001; visual mesh filename=package://boxygo_description/meshes/wheel.stl scale=0.001 0.001 0.001
- link right_wheel_2: geometry collision mesh filename=package://boxygo_description/meshes/wheel.dae scale=0.001 0.001 0.001; visual mesh filename=package://boxygo_description/meshes/wheel.stl scale=0.001 0.001 0.001
- link right_wheel_3: geometry collision mesh filename=package://boxygo_description/meshes/wheel.dae scale=0.001 0.001 0.001; visual mesh filename=package://boxygo_description/meshes/wheel.stl scale=0.001 0.001 0.001
