Commit message: urdf update

File: src/boxygo_description/urdf/common/lidar.xacro (robot description, xacro)
@@ -5,5 +5,5 @@
       <parent link="${parent_link}"/>
       <child link="laser_frame"/>
-      <origin xyz="${x_offset} ${y_offset} ${z_offset}" rpy="0 0 0"/>
+      <origin xyz="${x_offset} ${y_offset} ${z_offset}" rpy="0 0 ${-math.pi/2}"/>
     </joint>
     <link name="laser_frame">

File: src/boxygo_description/urdf/common/robot_joints.xacro (robot description, xacro)
@@ -1,19 +1,29 @@
 <?xml version="1.0"?>
 <robot xmlns:xacro="http://ros.org/wiki/xacro">
-  <joint name="right_rocker_beam_joint" type="revolute">
+  <xacro:arg name="sim_mode" default="gazebo"/>
+  <xacro:property name="sim_mode_prop" value="$(arg sim_mode)"/>
+  <xacro:property name="rocker_joint_type" value="revolute"/>
+  <xacro:if value="${sim_mode_prop == 'real'}">
+    <xacro:property name="rocker_joint_type" value="fixed"/>
+  </xacro:if>
+  <joint name="right_rocker_beam_joint" type="${rocker_joint_type}">
     <parent link="base_link"/>
     <child link="right_rocker_beam"/>
     <origin xyz="${rocker_x_offset} ${-rocker_y_offset} ${rocker_z_offset}" rpy="0 0 0"/>
     <axis xyz="0 1 0"/>
-    <limit lower="${-math.pi/12}" upper="${math.pi/12}" effort="50.0" velocity="10.0"/>
-    <dynamics damping="0.05" friction="0.005"/>
+    <xacro:if value="${rocker_joint_type != 'fixed'}">
+      <limit lower="${-math.pi/12}" upper="${math.pi/12}" effort="50.0" velocity="10.0"/>
+      <dynamics damping="0.05" friction="0.005"/>
+    </xacro:if>
   </joint>
-  <joint name="left_rocker_beam_joint" type="revolute">
+  <joint name="left_rocker_beam_joint" type="${rocker_joint_type}">
     <parent link="base_link"/>
     <child link="left_rocker_beam"/>
     <origin xyz="${rocker_x_offset} ${rocker_y_offset} ${rocker_z_offset}" rpy="0 0 ${math.pi}"/>
     <axis xyz="0 1 0"/>
-    <limit lower="${-math.pi/12}" upper="${math.pi/12}" effort="50.0" velocity="10.0"/>
-    <dynamics damping="0.05" friction="0.005"/>
+    <xacro:if value="${rocker_joint_type != 'fixed'}">
+      <limit lower="${-math.pi/12}" upper="${math.pi/12}" effort="50.0" velocity="10.0"/>
+      <dynamics damping="0.05" friction="0.005"/>
+    </xacro:if>
   </joint>
   <xacro:macro name="wheel_assembly" params="side parent_link sign wheel_side_sign index x_offset y_offset z_offset">

Commit message: add position reset

File: src/boxygo_description/urdf/common/lidar.xacro (robot description, xacro)
@@ -5,5 +5,9 @@
       <parent link="${parent_link}"/>
       <child link="laser_frame"/>
+<<<<<<< HEAD
       <origin xyz="${x_offset} ${y_offset} ${z_offset}" rpy="0 0 ${-math.pi/2}"/>
+=======
+      <origin xyz="${x_offset} ${y_offset} ${z_offset}" rpy="0 0 ${pi}"/>
+>>>>>>> 52327ee (add position reset)
     </joint>
     <link name="laser_frame">

Commit message: rotate lidar

File: src/boxygo_description/urdf/common/lidar.xacro (robot description, xacro)
@@ -5,9 +5,5 @@
       <parent link="${parent_link}"/>
       <child link="laser_frame"/>
-<<<<<<< HEAD
-      <origin xyz="${x_offset} ${y_offset} ${z_offset}" rpy="0 0 ${-math.pi/2}"/>
-=======
       <origin xyz="${x_offset} ${y_offset} ${z_offset}" rpy="0 0 ${pi}"/>
->>>>>>> 52327ee (add position reset)
     </joint>
     <link name="laser_frame">

Commit message: update

File: src/boxygo_description/urdf/common/lidar.xacro (robot description, xacro)
@@ -5,5 +5,5 @@
       <parent link="${parent_link}"/>
       <child link="laser_frame"/>
-      <origin xyz="${x_offset} ${y_offset} ${z_offset}" rpy="0 0 ${pi}"/>
+      <origin xyz="${x_offset} ${y_offset} ${z_offset}" rpy="0 0 3.173"/>
     </joint>
     <link name="laser_frame">
@@ -30,9 +30,9 @@
       <sensor name="lidar" type="ray">
         <always_on>true</always_on>
-        <visualize>false</visualize> <update_rate>10</update_rate>
+        <visualize>false</visualize> <update_rate>8</update_rate>
         <ray>
           <scan>
             <horizontal>
-              <samples>360</samples>
+              <samples>560</samples>
               <resolution>1</resolution>
               <min_angle>-3.14</min_angle>
@@ -41,7 +41,7 @@
           </scan>
           <range>
-            <min>0.12</min>
+            <min>0.08</min>
             <max>12.0</max>
-            <resolution>0.015</resolution>
+            <resolution>0.0017</resolution>
           </range>
           <noise>

File: src/boxygo_description/urdf/config/gazebo.xacro (robot description, xacro)
@@ -48,5 +48,5 @@
   <gazebo>
     <plugin name="gazebo_ros2_control" filename="libgazebo_ros2_control.so">
-      <update_rate>60</update_rate>
+      <update_rate>30</update_rate>
       <parameters>$(find boxygo_controllers)/config/diff_drive_controller.yaml</parameters>
     </plugin>

File: src/boxygo_description/urdf/luksusowy_isaac.urdf (robot description, URDF)
Before this commit: robot delivery_robot, 24 links, 23 joints
Joints:
- joint laser_joint: origin xyz=0.06 0.0 0.32 rpy=0 0 3.141592653589793 -> xyz=0.06 0.0 0.32 rpy=0 0 3.173

File: src/boxygo_description/urdf/robot_luksusowy.urdf.xacro (robot description, xacro)
@@ -193,5 +193,5 @@
   <gazebo>
     <plugin name="gazebo_ros2_control" filename="libgazebo_ros2_control.so">
-      <update_rate>60</update_rate>
+      <update_rate>30</update_rate>
       <parameters>${boxygo_controllers_pkg}/config/diff_drive_controller.yaml</parameters>
     </plugin>

Commit message: add new lidar

File: src/boxygo_description/urdf/common/lidar.xacro (robot description, xacro)
@@ -5,5 +5,5 @@
       <parent link="${parent_link}"/>
       <child link="laser_frame"/>
-      <origin xyz="${x_offset} ${y_offset} ${z_offset}" rpy="0 0 3.173"/>
+      <origin xyz="${x_offset} ${y_offset} ${z_offset}" rpy="0 0 0"/> <!-- 3.173 -->
     </joint>
     <link name="laser_frame">

File: src/boxygo_description/urdf/luksusowy_isaac.urdf (robot description, URDF)
Before this commit: robot delivery_robot, 24 links, 23 joints
Joints:
- joint laser_joint: origin xyz=0.06 0.0 0.32 rpy=0 0 3.173 -> xyz=0.06 0.0 0.32 rpy=0 0 0
