Commit message: Update simulation, lidar, localization and nav2 configs
- tune diff_drive_controller and joy2twist params
- update lidar/gazebo URDF config and playground worlds (add playground_v2)
- replace playground_map with new playground map
- adjust mapping, nav2 nvblox MPPI params and rviz config
- bump ros2_controllers submodule

File: src/boxygo_description/urdf/common/lidar.xacro (robot description, xacro)
@@ -1,9 +1,9 @@
 <?xml version="1.0"?>
 <robot xmlns:xacro="http://ros.org/wiki/xacro">
-  <xacro:macro name="sensor_ydlidar" params="parent_link x_offset y_offset z_offset">
+  <xacro:macro name="sensor_hokuyo_ust10lx" params="parent_link x_offset y_offset z_offset">
     <joint name="laser_joint" type="fixed">
       <parent link="${parent_link}"/>
       <child link="laser_frame"/>
-      <origin xyz="${x_offset} ${y_offset} ${z_offset}" rpy="0 0 3.173"/>
+      <origin xyz="${x_offset} ${y_offset} ${z_offset}" rpy="0 0 0"/>
     </joint>
     <link name="laser_frame">
@@ -28,20 +28,21 @@
     </link>
     <gazebo reference="laser_frame">
-      <sensor name="lidar" type="ray">
+      <sensor name="ust_10lx" type="ray">
         <always_on>true</always_on>
-        <visualize>false</visualize> <update_rate>8</update_rate>
+        <visualize>false</visualize>
+        <update_rate>40</update_rate>
         <ray>
           <scan>
             <horizontal>
-              <samples>560</samples>
+              <samples>1081</samples>
               <resolution>1</resolution>
-              <min_angle>-3.14</min_angle>
-              <max_angle>3.14</max_angle>
+              <min_angle>-2.35619449</min_angle>
+              <max_angle>2.35619449</max_angle>
             </horizontal>
           </scan>
           <range>
-            <min>0.08</min>
-            <max>12.0</max>
-            <resolution>0.0017</resolution>
+            <min>0.04</min>
+            <max>10.0</max>
+            <resolution>0.01</resolution>
           </range>
           <noise>

File: src/boxygo_description/urdf/luksusowy.urdf.xacro (robot description, xacro)
@@ -14,6 +14,6 @@
   </xacro:if>
   <xacro:include filename="$(find boxygo_description)/urdf/common/lidar.xacro"/>
-  <xacro:include filename="$(find boxygo_description)/urdf/common/_d435i.urdf.xacro"/>
-  <xacro:sensor_ydlidar parent_link="base_link" x_offset="0.06" y_offset="0.0" z_offset="0.32"/>
-  <xacro:sensor_d435i parent="base_link" use_nominal_extrinsics="true"> <origin xyz="0.38 0.0 0.225" rpy="0 0 0"/></xacro:sensor_d435i>
+  <!-- <xacro:include filename="$(find boxygo_description)/urdf/common/_d435i.urdf.xacro"/> -->
+  <xacro:sensor_hokuyo_ust10lx parent_link="base_link" x_offset="0.06" y_offset="0.0" z_offset="0.32"/>
+  <!-- <xacro:sensor_d435i parent="base_link" use_nominal_extrinsics="true"> <origin xyz="0.38 0.0 0.225" rpy="0 0 0"/></xacro:sensor_d435i> -->
 </robot>

File: src/boxygo_description/urdf/luksusowy_isaac.urdf (robot description, URDF)
Before this commit: robot delivery_robot, 24 links, 23 joints
Links:
- removed link camera_accel_frame
- removed link camera_accel_optical_frame
- removed link camera_bottom_screw_frame
- removed link camera_color_frame
- removed link camera_color_optical_frame
- removed link camera_depth_frame
- removed link camera_depth_optical_frame
- removed link camera_gyro_frame
- removed link camera_gyro_optical_frame
- removed link camera_infra1_frame
- removed link camera_infra1_optical_frame
- removed link camera_infra2_frame
- removed link camera_infra2_optical_frame
- removed link camera_link
Joints:
- removed joint camera_accel_joint
- removed joint camera_accel_optical_joint
- removed joint camera_color_joint
- removed joint camera_color_optical_joint
- removed joint camera_depth_joint
- removed joint camera_depth_optical_joint
- removed joint camera_gyro_joint
- removed joint camera_gyro_optical_joint
- removed joint camera_infra1_joint
- removed joint camera_infra1_optical_joint
- removed joint camera_infra2_joint
- removed joint camera_infra2_optical_joint
- removed joint camera_joint
- removed joint camera_link_joint
- joint laser_joint: origin xyz=0.06 0.0 0.32 rpy=0 0 3.173 -> xyz=0.06 0.0 0.32 rpy=0 0 0
